Commit message: added colored blocks

File: spinner_description/urdf/materials.xacro (robot description, xacro)
@@ -25,6 +25,15 @@
     <color rgba="0.8 0.0 0.0 1.0"/>
   </material>
+  <material name="yellow">
+    <color rgba="0.6 0.6 0.0 1.0"/>
+  </material>
   <material name="white">
     <color rgba="1.0 1.0 1.0 1.0"/>
   </material>
+  <material name="whorl">
+    <texture filename="package://spinner_description/materials/textures/barrelgradient.png" />
+  </material>
+  <material name="squares">
+    <texture filename="package://spinner_description/materials/textures/squares.png" />
+  </material>
 </robot>

File: spinner_description/urdf/spinner.urdf (robot description, URDF)
Before this commit: robot spinner, 6 links, 5 joints
Links:
- added link black_blk, mass 0.01; collision box size=0.1 0.1 0.1; visual box size=0.1 0.1 0.1
- added link blue_blk, mass 0.01; collision box size=0.1 0.1 0.1; visual box size=0.1 0.1 0.1
- added link green_blk, mass 0.01; collision box size=0.1 0.1 0.1; visual box size=0.1 0.1 0.1
- added link orange_blk, mass 0.01; collision box size=0.1 0.1 0.1; visual box size=0.1 0.1 0.1
- added link red_blk, mass 0.01; collision box size=0.1 0.1 0.1; visual box size=0.1 0.1 0.1
- added link yellow_blk, mass 0.01; collision box size=0.1 0.1 0.1; visual box size=0.1 0.1 0.1
- link camera_link: mass 1 -> 0.01
Joints:
- removed joint polecam
- added joint black_jt: type fixed, parent barrel, child black_blk, origin xyz=-0.25 -0.42 0 rpy=0 0 0
- added joint blue_jt: type fixed, parent barrel, child blue_blk, origin xyz=0.5 0 0 rpy=0 0 0
- added joint green_jt: type fixed, parent barrel, child green_blk, origin xyz=-0.5 0 0 rpy=0 0 0
- added joint orange_jt: type fixed, parent barrel, child orange_blk, origin xyz=0.25 -0.42 0 rpy=0 0 0
- added joint pancam: type revolute, parent pole, child camera_link, origin xyz=0 0 2.0 rpy=0 0 0, axis 0 0 1, limit lower=-0.1 upper=0.1 effort=1000 velocity=0.5
- added joint red_jt: type fixed, parent barrel, child red_blk, origin xyz=0.25 0.42 0 rpy=0 0 0
- added joint yellow_jt: type fixed, parent barrel, child yellow_blk, origin xyz=-0.25 0.42 0 rpy=0 0 0

File: spinner_description/urdf/spinner.urdf.xacro (robot description, xacro)
@@ -71,11 +71,20 @@
     </inertial>
   </link>
-  <joint name="polecam" type="fixed">
+    <!--limit effort="1000" lower="-1" upper="1" velocity="0.5"/-->
+  <joint name="pancam" type="revolute">
     <parent link="pole"/>
     <child link="camera_link"/>
-  </joint>
+    <origin xyz="0 0 2.0" rpy="0 0 0"/>
+    <axis xyz="0 0 1"/>
+    <limit effort="1000" lower="-0.1" upper="0.1" velocity="0.5"/>
+    <dynamics damping="0.7"/>
+  </joint>
+  <!--joint name="polecam" type="fixed">
+    <parent link="pole"/>
+    <child link="camera_link"/>
+  </joint-->
   <link name="camera_link">
     <collision>
-      <origin xyz="0 0 2.0" rpy="1.5707 0 0"/>
+      <origin xyz="0 0 0" rpy="0 0 0"/>
       <geometry>
 	<box size="0.1 0.1 0.1"/>
@@ -83,5 +92,5 @@
     </collision>
     <visual>
-      <origin xyz="0 0 2.0" rpy="0 0 0"/>
+      <origin xyz="0 0 0" rpy="0 0 0"/>
       <geometry>
 	<box size="0.1 0.1 0.1"/>
@@ -90,6 +99,6 @@
     </visual>
     <inertial>
-      <origin xyz="0 0 0" rpy="0 0 1.5707"/>
-      <mass value="1"/>
+      <origin xyz="0 0 0" rpy="0 0 0"/>
+      <mass value="0.01"/>
       <inertia
 	  ixx="1" ixy="0.0" ixz="0.0"
@@ -158,5 +167,5 @@
     <origin xyz="0 0 2.0" rpy="0 0 0"/>
     <axis xyz="0 0 1"/>
-    <dynamics damping="0.7"/>
+    <dynamics damping="10.0"/>
   </joint>
   <joint name="elevation" type="continuous">
@@ -165,5 +174,5 @@
     <origin xyz="0 0 0" rpy="0 0 0"/>
     <axis xyz="1 0 0"/>
-    <dynamics damping="0.7"/>
+    <dynamics damping="10.0"/>
   </joint>
   <joint name="spinner" type="continuous">
@@ -172,5 +181,5 @@
     <origin xyz="0 1.0 0" rpy="0 0 0"/>
     <axis xyz="0 0 1"/>
-    <dynamics damping="0.7"/>
+    <dynamics damping="1.0"/>
   </joint>
   <link name="arm">
@@ -209,5 +218,6 @@
 	<cylinder radius="0.5" length="0.1"/>
       </geometry>
-      <material name="orange"/>
+      <!--material name="orange"/-->
+      <material name="whorl"/>
     </visual>
     <inertial>
@@ -220,3 +230,45 @@
     </inertial>
   </link>
+  <link name="blue_blk">
+    <collision><geometry><box size="0.1 0.1 0.1"/></geometry></collision>
+    <visual><geometry><box size="0.1 0.1 0.1"/></geometry><material name="blue"/></visual>
+    <inertial><mass value="0.01"/><inertia ixx="1" ixy="0.0" ixz="0.0" iyy="1"
+       iyz="0.0" izz="1"/></inertial></link>
+  <joint name="blue_jt" type="fixed"><parent link="barrel"/><child link="blue_blk"/>
+    <origin xyz="0.5 0 0" rpy="0 0 0"/></joint>
+  <link name="red_blk">
+    <collision><geometry><box size="0.1 0.1 0.1"/></geometry></collision>
+    <visual><geometry><box size="0.1 0.1 0.1"/></geometry><material name="red"/></visual>
+    <inertial><mass value="0.01"/><inertia ixx="1" ixy="0.0" ixz="0.0" iyy="1"
+       iyz="0.0" izz="1"/></inertial></link>
+  <joint name="red_jt" type="fixed"><parent link="barrel"/><child link="red_blk"/>
+    <origin xyz="0.25 0.42 0" rpy="0 0 0"/></joint>
+  <link name="yellow_blk">
+    <collision><geometry><box size="0.1 0.1 0.1"/></geometry></collision>
+    <visual><geometry><box size="0.1 0.1 0.1"/></geometry><material name="yellow"/></visual>
+    <inertial><mass value="0.01"/><inertia ixx="1" ixy="0.0" ixz="0.0" iyy="1"
+       iyz="0.0" izz="1"/></inertial></link>
+  <joint name="yellow_jt" type="fixed"><parent link="barrel"/><child link="yellow_blk"/>
+    <origin xyz="-0.25 0.42 0" rpy="0 0 0"/></joint>
+  <link name="green_blk">
+    <collision><geometry><box size="0.1 0.1 0.1"/></geometry></collision>
+    <visual><geometry><box size="0.1 0.1 0.1"/></geometry><material name="green"/></visual>
+    <inertial><mass value="0.01"/><inertia ixx="1" ixy="0.0" ixz="0.0" iyy="1"
+       iyz="0.0" izz="1"/></inertial></link>
+  <joint name="green_jt" type="fixed"><parent link="barrel"/><child link="green_blk"/>
+    <origin xyz="-0.5 0 0" rpy="0 0 0"/></joint>
+  <link name="black_blk">
+    <collision><geometry><box size="0.1 0.1 0.1"/></geometry></collision>
+    <visual><geometry><box size="0.1 0.1 0.1"/></geometry><material name="black"/></visual>
+    <inertial><mass value="0.01"/><inertia ixx="1" ixy="0.0" ixz="0.0" iyy="1"
+       iyz="0.0" izz="1"/></inertial></link>
+  <joint name="black_jt" type="fixed"><parent link="barrel"/><child link="black_blk"/>
+    <origin xyz="-0.25 -0.42 0" rpy="0 0 0"/></joint>
+  <link name="orange_blk">
+    <collision><geometry><box size="0.1 0.1 0.1"/></geometry></collision>
+    <visual><geometry><box size="0.1 0.1 0.1"/></geometry><material name="orange"/></visual>
+    <inertial><mass value="0.01"/><inertia ixx="1" ixy="0.0" ixz="0.0" iyy="1"
+       iyz="0.0" izz="1"/></inertial></link>
+  <joint name="orange_jt" type="fixed"><parent link="barrel"/><child link="orange_blk"/>
+    <origin xyz="0.25 -0.42 0" rpy="0 0 0"/></joint>
 </robot>
